File: pcbs/bme680sensor.kicad_sch (KiCad schematic)
At the start: 3 parts, among them J10 Conn_01x04_Pin, U6 BME680

Commit message: try to fix kicad weirdness
Parts:
- renumbered U6 to U7
Changed lines of the file:
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@@
 		(in_pos_files yes)
 		(dnp no)
-		(property "Reference" "U6"
+		(property "Reference" "U7"
 			(at 139.7 62.2301 0)
 			(show_name no)
@@
 			(project "monstera"
 				(path "/9190de51-0203-4be2-9542-a4d25603b986"
-					(reference "U6")
+					(reference "U7")
 					(unit 1)
 				)

Commit message: make sensor pcbs
Parts:
- removed U7: BME680, Package_LGA:Bosch_LGA-8_3x3mm_P0.8mm_ClockwisePinNumbering, symbol Sensor:BME680
- added H1, H2, H3, H4: MountingHole, symbol Mechanical:MountingHole
- added U1: BME680_Breakout, Aloe:BME680_Breakout_Board, symbol Aloe:BME680_Breakout
- J10: footprint (none) -> Connector_JST:JST_PH_S4B-PH-K_1x04_P2.00mm_Horizontal
- JP1: footprint (none) -> Jumper:SolderJumper-3_P1.3mm_Bridged12_RoundedPad1.0x1.5mm
Connections:
- net +3V3: now also U1.1 (VCC), U1.6 (CSB)
- net GND: now also U1.2 (GND)
- net I2CSCL: now also U1.3 (SCK)
- net I2CSDA: now also U1.4 (SDI)
- net at JP1.2 (C): now also U1.5 (SDO)
