File: pcbs/reedsensor/reedsensor.kicad_pcb (KiCad board)
At the start: 2 copper layers, 21.6 x 17.8 mm, 9 parts, among them J9 Conn_01x03_Pin, SW1 SW_Reed, U6 DRV5033AJxLPG

Commit message: reed and hall effect sensor, test gerber files (not ready for production)
Parts:
- C1: renamed from C2; value ~ -> 680pF
- renumbered J9 to J1, R4 to R1, U6 to U1
Changed lines of the file:
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@@
 			(size 2.5 2)
 			(layers "F.Cu" "F.Mask" "F.Paste")
-			(net "Net-(J9-Pin_3)")
+			(net "Net-(J1-Pin_3)")
 			(pinfunction "2_2")
 			(pintype "passive")
@@
 		(descr "Capacitor SMD 0805 (2012 Metric), square (rectangular) end terminal, IPC-7351 nominal with elongated pad for handsoldering. (Body size source: IPC-SM-782 page 76, https://www.pcb-3d.com/wordpress/wp-content/uploads/ipc-sm-782a_amendment_1_and_2.pdf, https://docs.google.com/spreadsheets/d/1BsfQQcO9C6DZCsRaXUlFlo91Tg2WpOkGARC1WS5S8t0/edit?usp=sharing)")
 		(tags "capacitor handsolder")
-		(property "Reference" "C2"
+		(property "Reference" "C1"
 			(at -3.175 0 0)
 			(layer "F.SilkS")
@@
 			)
 		)
-		(property "Value" "~"
+		(property "Value" "680pF"
 			(at 0 1.68 0)
 			(layer "F.Fab")
@@
 				(font
 					(size 1.27 1.27)
-				)
-			)
-		)
-		(property "KiLib_Generator" "SMD_2terminal_chip_molded"
-			(at 0 0 0)
-			(layer "F.SilkS")
-			(hide yes)
-			(effects
-				(font
-					(size 1 1)
-					(thickness 0.15)
 				)
 			)
@@
 		(descr "Resistor SMD 0805 (2012 Metric), square (rectangular) end terminal, IPC-7351 nominal with elongated pad for handsoldering. (Body size source: IPC-SM-782 page 72, https://www.pcb-3d.com/wordpress/wp-content/uploads/ipc-sm-782a_amendment_1_and_2.pdf)")
 		(tags "resistor handsolder")
-		(property "Reference" "R4"
+		(property "Reference" "R1"
 			(at 3.175 0.635 0)
 			(layer "F.SilkS")
@@
 				(font
 					(size 1.27 1.27)
-				)
-			)
-		)
-		(property "KiLib_Generator" "SMD_2terminal_chip_molded"
-			(at 0 0 0)
-			(layer "F.SilkS")
-			(hide yes)
-			(effects
-				(font
-					(size 1 1)
-					(thickness 0.15)
 				)
 			)
@@
 			(layers "F.Cu" "F.Mask" "F.Paste")
 			(roundrect_rratio 0.208333)
-			(net "Net-(J9-Pin_3)")
+			(net "Net-(J1-Pin_3)")
 			(pintype "passive")
 		)
@@
 				(font
 					(size 1.27 1.27)
-				)
-			)
-		)
-		(property "KiLib_Generator" "mounting_hardware/mounting_hole"
-			(at 0 0 0)
-			(layer "F.SilkS")
-			(hide yes)
-			(effects
-				(font
-					(size 1 1)
-					(thickness 0.15)
 				)
 			)
@@
 		(descr "JST PH series connector, S3B-PH-K (http://www.jst-mfg.com/product/pdf/eng/ePH.pdf)")
 		(tags "connector JST PH horizontal")
-		(property "Reference" "J9"
+		(property "Reference" "J1"
 			(at -3.715 0.635 0)
 			(layer "F.SilkS")
@@
 				(font
 					(size 1.27 1.27)
-				)
-			)
-		)
-		(property "KiLib_Generator" "connector/JST"
-			(at 0 0 0)
-			(layer "F.SilkS")
-			(hide yes)
-			(effects
-				(font
-					(size 1 1)
-					(thickness 0.15)
 				)
 			)
@@
 			(layers "*.Cu" "*.Mask")
 			(remove_unused_layers no)
-			(net "Net-(J9-Pin_3)")
+			(net "Net-(J1-Pin_3)")
 			(pinfunction "Pin_3_3")
 			(pintype "passive")
@@
 				(font
 					(size 1.27 1.27)
-				)
-			)
-		)
-		(property "KiLib_Generator" "mounting_hardware/mounting_hole"
-			(at 0 0 0)
-			(layer "F.SilkS")
-			(hide yes)
-			(effects
-				(font
-					(size 1 1)
-					(thickness 0.15)
 				)
 			)
@@
 			)
 		)
-		(property "KiLib_Generator" "mounting_hardware/mounting_hole"
-			(at 0 0 0)
-			(layer "F.SilkS")
-			(hide yes)
-			(effects
-				(font
-					(size 1 1)
-					(thickness 0.15)
-				)
-			)
-		)
 		(property ki_fp_filters "MountingHole*")
 		(sheetname "/")
@@
 			)
 		)
-		(property "KiLib_Generator" "mounting_hardware/mounting_hole"
-			(at 0 0 0)
-			(layer "F.SilkS")
-			(hide yes)
-			(effects
-				(font
-					(size 1 1)
-					(thickness 0.15)
-				)
-			)
-		)
 		(property ki_fp_filters "MountingHole*")
 		(sheetname "/")
@@
 		(descr "TO-92 leads in-line, narrow, oval pads, drill 0.75mm (see NXP sot054_po.pdf)")
 		(tags "to-92 sc-43 sc-43a sot54 PA33 transistor")
-		(property "Reference" "U6"
+		(property "Reference" "U1"
 			(at -2.54 -1.905 0)
 			(layer "F.SilkS")
@@
 		(property ki_fp_filters "TO?92*")
 		(sheetname "/")
-		(sheetfile "halleffectsimplesensor.kicad_sch")
+		(sheetfile "reedsensor.kicad_sch")
+		(units
+			(unit
+				(name "A")
+				(pins "1" "2" "3")
+			)
+		)
 		(attr through_hole)
 		(duplicate_pad_numbers_are_jumpers no)
@@
 			(layers "*.Cu" "*.Mask")
 			(remove_unused_layers no)
-			(net "Net-(J9-Pin_3)")
+			(net "Net-(J1-Pin_3)")
 			(pinfunction "OUT_3")
 			(pintype "output")
@@
 		(width 0.2)
 		(layer "F.Cu")
-		(net "Net-(J9-Pin_3)")
+		(net "Net-(J1-Pin_3)")
 	)
 	(segment
@@
 		(width 0.2)
 		(layer "F.Cu")
-		(net "Net-(J9-Pin_3)")
+		(net "Net-(J1-Pin_3)")
 	)
 	(segment
@@
 		(width 0.2)
 		(layer "F.Cu")
-		(net "Net-(J9-Pin_3)")
+		(net "Net-(J1-Pin_3)")
 	)
 	(segment
@@
 		(width 0.2)
 		(layer "F.Cu")
-		(net "Net-(J9-Pin_3)")
+		(net "Net-(J1-Pin_3)")
 	)
 	(segment
@@
 		(width 0.2)
 		(layer "F.Cu")
-		(net "Net-(J9-Pin_3)")
+		(net "Net-(J1-Pin_3)")
 	)
 	(segment
@@
 		(width 0.2)
 		(layer "F.Cu")
-		(net "Net-(J9-Pin_3)")
+		(net "Net-(J1-Pin_3)")
 	)
 	(zone
