File: pcbs/reedsensor/reedsensor.kicad_sch (KiCad schematic)
At the start: 8 parts, among them J9 Conn_01x03_Pin, SW1 SW_Reed

Commit message: reed and hall effect sensor, test gerber files (not ready for production)
Parts:
- added U1: DRV5033AJxLPG, Package_TO_SOT_THT:TO-92_Inline, symbol Sensor_Magnetic:DRV5033AJxLPG
- C1: renamed from C2; value (none) -> 680pF
- renumbered J9 to J1, R4 to R1
Connections:
- net +3V3: now also U1.1 (VCC)
- net GND: now also U1.2 (GND)
- net at J1.3 (Pin_3), R1.2, SW1.2: now also U1.3 (OUT)
Changed lines of the file:
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@@
 	(paper "A4")
+	(junction
+		(at 132.08 64.77)
+		(diameter 0)
+		(color 0 0 0 0)
+	)
 	(junction
 		(at 88.9 59.69)
@@
 	)
 	(junction
+		(at 113.03 53.34)
+		(diameter 0)
+		(color 0 0 0 0)
+	)
+	(junction
 		(at 91.44 76.2)
 		(diameter 0)
@@
 		(color 0 0 0 0)
 	)
+	(junction
+		(at 132.08 76.2)
+		(diameter 0)
+		(color 0 0 0 0)
+	)
+	(wire
+		(pts
+			(xy 132.08 64.77) (xy 148.59 64.77)
+		)
+		(stroke
+			(width 0)
+			(type default)
+		)
+	)
 	(wire
 		(pts
@@
 	(wire
 		(pts
+			(xy 158.75 54.61) (xy 158.75 53.34)
+		)
+		(stroke
+			(width 0)
+			(type default)
+		)
+	)
+	(wire
+		(pts
 			(xy 85.09 53.34) (xy 88.9 53.34)
 		)
@@
 	(wire
 		(pts
+			(xy 113.03 53.34) (xy 158.75 53.34)
+		)
+		(stroke
+			(width 0)
+			(type default)
+		)
+	)
+	(wire
+		(pts
+			(xy 132.08 76.2) (xy 158.75 76.2)
+		)
+		(stroke
+			(width 0)
+			(type default)
+		)
+	)
+	(wire
+		(pts
 			(xy 72.39 64.77) (xy 113.03 64.77)
 		)
@@
 		(pts
 			(xy 88.9 53.34) (xy 88.9 54.61)
+		)
+		(stroke
+			(width 0)
+			(type default)
+		)
+	)
+	(wire
+		(pts
+			(xy 158.75 74.93) (xy 158.75 76.2)
 		)
 		(stroke
@@
 		(dnp no)
 		(fields_autoplaced yes)
-		(property "Reference" "#PWR019"
+		(property "Reference" "#PWR02"
 			(at 91.44 88.9 0)
 			(hide yes)
@@
 			(project "reedsensor"
 				(path "/ce879ccc-6552-4813-89f0-266e598c9a4a"
-					(reference "#PWR019")
+					(reference "#PWR02")
 					(unit 1)
 				)
@@
 		(dnp no)
 		(fields_autoplaced yes)
-		(property "Reference" "R4"
+		(property "Reference" "R1"
 			(at 115.57 57.1499 0)
 			(show_name no)
@@
 			(project "reedsensor"
 				(path "/ce879ccc-6552-4813-89f0-266e598c9a4a"
-					(reference "R4")
+					(reference "R1")
 					(unit 1)
 				)
@@
 		(dnp no)
 		(fields_autoplaced yes)
-		(property "Reference" "#PWR018"
+		(property "Reference" "#PWR01"
 			(at 85.09 53.34 0)
 			(hide yes)
@@
 			(project "reedsensor"
 				(path "/ce879ccc-6552-4813-89f0-266e598c9a4a"
-					(reference "#PWR018")
+					(reference "#PWR01")
 					(unit 1)
 				)
@@
 		(dnp no)
 		(fields_autoplaced yes)
-		(property "Reference" "J9"
+		(property "Reference" "J1"
 			(at 67.945 54.61 0)
 			(show_name no)
@@
 			(project "reedsensor"
 				(path "/ce879ccc-6552-4813-89f0-266e598c9a4a"
-					(reference "J9")
+					(reference "J1")
 					(unit 1)
 				)
@@
 		(dnp no)
 		(fields_autoplaced yes)
-		(property "Reference" "C2"
+		(property "Reference" "C1"
 			(at 91.44 57.1562 0)
 			(show_name no)
@@
 			)
 		)
-		(property "Value" ""
+		(property "Value" "680pF"
 			(at 91.44 58.4262 0)
 			(show_name no)
@@
 			(project "reedsensor"
 				(path "/ce879ccc-6552-4813-89f0-266e598c9a4a"
-					(reference "C2")
+					(reference "C1")
 					(unit 1)
 				)
@@
 					(unit 1)
 				)
+			)
+		)
+	)
+	(symbol
+		(lib_id "Sensor_Magnetic:DRV5033AJxLPG")
+		(at 156.21 64.77 0)
+		(mirror y)
+		(unit 1)
+		(body_style 1)
+		(exclude_from_sim no)
+		(in_bom yes)
+		(on_board yes)
+		(in_pos_files yes)
+		(dnp no)
+		(fields_autoplaced yes)
+		(property "Reference" "U1"
+			(at 162.56 63.4999 0)
+			(show_name no)
+			(do_not_autoplace no)
+			(effects
+				(font
+					(size 1.27 1.27)
+				)
+				(justify right)
+			)
+		)
+		(property "Value" "DRV5033AJxLPG"
+			(at 162.56 66.0399 0)
+			(show_name no)
+			(do_not_autoplace no)
+			(effects
+				(font
+					(size 1.27 1.27)
+				)
+				(justify right)
+			)
+		)
+		(property "Footprint" "Package_TO_SOT_THT:TO-92_Inline"
+			(at 156.21 64.77 0)
+			(hide yes)
+			(show_name no)
+			(do_not_autoplace no)
+			(effects
+				(font
+					(size 1.27 1.27)
+				)
+			)
+		)
+		(property "Datasheet" "https://www.ti.com/lit/ds/symlink/drv5033.pdf"
+			(at 156.21 64.77 0)
+			(hide yes)
+			(show_name no)
+			(do_not_autoplace no)
+			(effects
+				(font
+					(size 1.27 1.27)
+				)
+			)
+		)
+		(property "Description" "±6.9 / ±3.5 mT, 20-kHz, 2-38V, TO-92"
+			(at 156.21 64.77 0)
+			(hide yes)
+			(show_name no)
+			(do_not_autoplace no)
+			(effects
+				(font
+					(size 1.27 1.27)
+				)
+			)
+		)
+		(pin "1"
+		)
+		(pin "3"
+		)
+		(pin "2"
+		)
+		(instances
+			(project "reedsensor"
+				(path "/ce879ccc-6552-4813-89f0-266e598c9a4a"
+					(reference "U1")
+					(unit 1)
+				)
